File: PCB/PCB.sch (KiCad schematic (older format))
At the start: 21 parts

Commit message: Add files via upload
Parts:
- added U?: KY-037, symbol KY-037:KY-037
Changed lines of the file:
@@
 Text GLabel 3800 6050 2    50   Input ~ 0
 5V
+$Comp
+L KY-037:KY-037 U?
+U 1 1 600128CD
+P 2950 6150
+F 0 "U?" H 3000 6600 50  0000 L CNN
+F 1 "KY-037" H 2900 6500 50  0000 L CNN
+F 2 "" H 2950 6150 50  0001 C CNN
+F 3 "" H 2950 6150 50  0001 C CNN
+	1    2950 6150
+	1    0    0    -1
+$EndComp
 $EndSCHEMATC
